File: control.brd (EAGLE design)
At the start: 100 x 80 mm, 21 parts, among them IC1 OPA336P, Q1 BSS92, Q2 BSS101

Commit message: +added main discharge path
Parts:
- added JP5: (no value), jumper:JP4
- added R14, R15: (no value), resistor:M0805
- added R16, R17: (no value), resistor-power:RS02M
- added U$3: STL100NH3LL, teile:PG-TDSON-8
Connections:
- new net ADC4: JP3.1, JP5.4, R13.1, R15.2, R17.2, R2.2
- new net N$14: JP5.1, R16.1, U$3.5, U$3.6, U$3.7, U$3.8, U$3.TH
- new net N$15: JP5.3, R16.2
- new net N$16: JP5.2, R17.1
- net GND: now also R14.1
- net N$10: now also R14.2, R15.1; no longer JP3.1, R13.1, R2.2
Routing:
- net N$10: track 37.8 -> 0.00 mm
- net ADC4: track 0.00 -> 37.8 mm
- net N$9: track 18.0 -> 14.3 mm
Other:
- outline, holes or cut-outs redrawn
Changed lines of the file:
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@@
 <setting verticaltext="up"/>
 </settings>
-<grid distance="0.05" unitdist="inch" unit="inch" style="lines" multiple="2" display="yes" altdistance="0.025" altunitdist="inch" altunit="inch"/>
+<grid distance="1.27" unitdist="mm" unit="mm" style="lines" multiple="2" display="yes" altdistance="0.025" altunitdist="inch" altunit="inch"/>
 <layers>
 <layer number="1" name="Top" color="4" fill="1" visible="yes" active="yes"/>
@@
 <board>
 <plain>
-<wire x1="0" y1="0" x2="100" y2="0" width="0" layer="20"/>
+<wire x1="0" y1="0" x2="50" y2="0" width="0" layer="20"/>
+<wire x1="50" y1="0" x2="100" y2="0" width="0" layer="20"/>
 <wire x1="100" y1="0" x2="100" y2="80" width="0" layer="20"/>
-<wire x1="100" y1="80" x2="0" y2="80" width="0" layer="20"/>
+<wire x1="100" y1="80" x2="50" y2="80" width="0" layer="20"/>
+<wire x1="50" y1="80" x2="0" y2="80" width="0" layer="20"/>
 <wire x1="0" y1="80" x2="0" y2="0" width="0" layer="20"/>
+<wire x1="50" y1="0" x2="50" y2="80" width="0" layer="20"/>
 </plain>
 <attributes>
@@
 <attribute name="OC_FARNELL" value="unknown" x="49.53" y="57.15" size="1.778" layer="27" display="off"/>
 </element>
+<element name="JP5" library="jumper" package="JP4" value="" x="21.59" y="27.94" rot="R90"/>
+<element name="U$3" library="teile" package="PG-TDSON-8" value="STL100NH3LL" x="21.59" y="10.16" rot="R90"/>
+<element name="R16" library="resistor-power" package="RS02M" value="" x="25.4" y="27.94" rot="R90">
+<attribute name="OC_NEWARK" value="unknown" x="25.4" y="27.94" size="1.778" layer="27" rot="R90" display="off"/>
+<attribute name="MPN" value="" x="25.4" y="27.94" size="1.778" layer="27" rot="R90" display="off"/>
+<attribute name="MF" value="" x="25.4" y="27.94" size="1.778" layer="27" rot="R90" display="off"/>
+<attribute name="OC_FARNELL" value="unknown" x="25.4" y="27.94" size="1.778" layer="27" rot="R90" display="off"/>
+</element>
+<element name="R17" library="resistor-power" package="RS02M" value="" x="17.78" y="27.94" rot="R90">
+<attribute name="OC_NEWARK" value="unknown" x="17.78" y="27.94" size="1.778" layer="27" rot="R90" display="off"/>
+<attribute name="MPN" value="" x="17.78" y="27.94" size="1.778" layer="27" rot="R90" display="off"/>
+<attribute name="MF" value="" x="17.78" y="27.94" size="1.778" layer="27" rot="R90" display="off"/>
+<attribute name="OC_FARNELL" value="unknown" x="17.78" y="27.94" size="1.778" layer="27" rot="R90" display="off"/>
+</element>
+<element name="R14" library="resistor" package="M0805" value="" x="77.47" y="33.02"/>
+<element name="R15" library="resistor" package="M0805" value="" x="77.47" y="35.56"/>
 </elements>
 <signals>
@@
 </signal>
 <signal name="N$9">
+<contactref element="IC1" pad="6"/>
+<wire x1="60.96" y1="34.29" x2="60.96" y2="25.4" width="0.6096" layer="1"/>
+<wire x1="60.96" y1="25.4" x2="57.15" y2="21.59" width="0.6096" layer="1"/>
 <contactref element="Q1" pad="1"/>
 <contactref element="Q2" pad="2"/>
-<contactref element="IC1" pad="6"/>
-<wire x1="60.96" y1="29.21" x2="59.055" y2="29.21" width="0.6096" layer="1"/>
-<wire x1="59.69" y1="35.56" x2="60.96" y2="34.29" width="0.6096" layer="1"/>
-<wire x1="60.96" y1="34.29" x2="60.96" y2="29.21" width="0.6096" layer="1"/>
-<wire x1="60.96" y1="29.21" x2="60.96" y2="25.4" width="0.6096" layer="1"/>
-<wire x1="60.96" y1="25.4" x2="57.15" y2="21.59" width="0.6096" layer="1"/>
-</signal>
-<signal name="N$10">
-<contactref element="JP3" pad="1"/>
-<contactref element="R2" pad="2"/>
-<contactref element="R13" pad="1"/>
-<wire x1="33.02" y1="36.195" x2="30.48" y2="48.26" width="1.27" layer="1"/>
-<wire x1="30.48" y1="48.26" x2="34.29" y2="48.26" width="1.27" layer="1"/>
-<wire x1="34.29" y1="48.26" x2="36.83" y2="48.26" width="1.27" layer="1"/>
-<wire x1="36.83" y1="48.26" x2="38.1" y2="38.1" width="1.27" layer="1"/>
-<wire x1="34.29" y1="57.15" x2="34.29" y2="48.26" width="1.27" layer="1"/>
+<wire x1="60.96" y1="34.29" x2="59.69" y2="35.56" width="0" layer="19" extent="1-1"/>
+<wire x1="59.055" y1="29.21" x2="60.96" y2="25.4" width="0" layer="19" extent="1-1"/>
 </signal>
 <signal name="N$11">
@@
 <contactref element="U$1" pad="2"/>
 <contactref element="U$1" pad="3"/>
+<contactref element="R14" pad="1"/>
 <wire x1="70.17" y1="16.51" x2="70.17" y2="22.86" width="0" layer="19" extent="1-1"/>
 <wire x1="57.15" y1="19.05" x2="70.17" y2="16.51" width="0" layer="19" extent="1-1"/>
@@
 <wire x1="32.385" y1="7.435" x2="33.655" y2="7.435" width="0" layer="19" extent="1-1"/>
 <wire x1="46.67" y1="40.64" x2="57.15" y2="19.05" width="0" layer="19" extent="1-1"/>
+<wire x1="76.52" y1="33.02" x2="32.385" y2="7.435" width="0" layer="19" extent="1-1"/>
 </signal>
 <signal name="+12V">
@@
 <wire x1="72.07" y1="22.86" x2="72.07" y2="25.4" width="0" layer="19" extent="1-1"/>
 </signal>
+<signal name="N$14">
+<contactref element="U$3" pad="TH"/>
+<contactref element="U$3" pad="8"/>
+<contactref element="U$3" pad="5"/>
+<contactref element="U$3" pad="6"/>
+<contactref element="U$3" pad="7"/>
+<contactref element="JP5" pad="1"/>
+<contactref element="R16" pad="1"/>
+<wire x1="23.495" y1="12.985" x2="25.4" y2="18.415" width="0" layer="19" extent="1-1"/>
+<wire x1="22.225" y1="12.985" x2="23.495" y2="12.985" width="0" layer="19" extent="1-1"/>
+<wire x1="20.955" y1="12.985" x2="22.225" y2="12.985" width="0" layer="19" extent="1-1"/>
+<wire x1="19.685" y1="12.985" x2="20.955" y2="12.985" width="0" layer="19" extent="1-1"/>
+<wire x1="21.59" y1="10.885" x2="22.225" y2="12.985" width="0" layer="19" extent="1-1"/>
+<wire x1="21.59" y1="24.13" x2="23.495" y2="12.985" width="0" layer="19" extent="1-1"/>
+</signal>
+<signal name="N$15">
+<contactref element="R16" pad="2"/>
+<contactref element="JP5" pad="3"/>
+<wire x1="21.59" y1="29.21" x2="25.4" y2="37.465" width="0" layer="19" extent="1-1"/>
+</signal>
+<signal name="N$16">
+<contactref element="JP5" pad="2"/>
+<contactref element="R17" pad="1"/>
+<wire x1="21.59" y1="26.67" x2="17.78" y2="18.415" width="0" layer="19" extent="1-1"/>
+</signal>
+<signal name="ADC4">
+<contactref element="R15" pad="2"/>
+<contactref element="JP5" pad="4"/>
+<contactref element="R17" pad="2"/>
+<contactref element="JP3" pad="1"/>
+<contactref element="R2" pad="2"/>
+<contactref element="R13" pad="1"/>
+<wire x1="33.02" y1="36.195" x2="30.48" y2="48.26" width="1.27" layer="1"/>
+<wire x1="30.48" y1="48.26" x2="34.29" y2="48.26" width="1.27" layer="1"/>
+<wire x1="34.29" y1="48.26" x2="36.83" y2="48.26" width="1.27" layer="1"/>
+<wire x1="36.83" y1="48.26" x2="38.1" y2="38.1" width="1.27" layer="1"/>
+<wire x1="34.29" y1="57.15" x2="34.29" y2="48.26" width="1.27" layer="1"/>
+<wire x1="21.59" y1="31.75" x2="33.02" y2="36.195" width="0" layer="19" extent="1-1"/>
+<wire x1="17.78" y1="37.465" x2="21.59" y2="31.75" width="0" layer="19" extent="1-1"/>
+<wire x1="78.42" y1="35.56" x2="17.78" y2="37.465" width="0" layer="19" extent="1-1"/>
+</signal>
+<signal name="N$10">
+<contactref element="R15" pad="1"/>
+<contactref element="R14" pad="2"/>
+<wire x1="78.42" y1="33.02" x2="76.52" y2="35.56" width="0" layer="19" extent="1-1"/>
+</signal>
 </signals>

Commit message: +µC
Parts:
- removed R13: (no value), resistor-power:RWM5X26
- added C1, C2, C3, C4, C5, C6: (no value), resistor:C0805K
- added IC2: XMEGA16A4A, atmel:TQFP44
- added IC3: LM317MBSTT3, v-reg:SOT223
- added JP4, JP6: (no value), jumper:JP4
- added R18, R19, R20: (no value), resistor:M0805
Connections:
- new net +3V3: C1.1, C2.1, C3.1, C4.1, C5.1, IC2.19, IC2.31, IC2.39, IC2.9, IC3.4, R18.2, R20.2
- new net N$17: IC2.35, R18.1
- new net N$18: IC2.40, JP6.4
- new net N$19: IC2.41, JP6.3
- new net N$20: IC2.42, JP6.2
- new net N$21: IC2.43, JP6.1
- new net N$22: IC2.44, JP4.4
- new net N$23: IC2.1, JP4.3
- new net N$24: IC2.2, JP4.2
- new net N$25: IC2.3, JP4.1
- new net N$27: IC3.1, R19.2, R20.1
- net +12V: now also C6.1, IC3.3; no longer R13.2
- net ADC4: no longer R13.1
- net GND: now also C1.2, C2.2, C3.2, C4.2, C5.2, C6.2, IC2.18, IC2.30, IC2.38, IC2.8, R19.1
Routing:
- net ADC4: track 37.8 -> 0.00 mm

Commit message: +spannungsregler
Parts:
- added C7, C8: (no value), resistor:C0805K
- added IC4: OPA336P, burr-brown:DIL08
- added Q5: TIP41C, transistor-power:TO220AV
- added Q6: TIP42C, transistor-power:TO220AV
- added Q7: BC338, transistor-npn:TO92-EBC
- added R13, R21, R22: (no value), resistor:M0805
Connections:
- new net N$12: C7.1, Q5.E, R22.1
- new net N$13: Q7.C, R13.2
- new net N$26: Q6.B, R13.1
- new net N$28: C8.1, IC4.6, Q7.B
- new net N$30: C8.2, IC4.2, R21.1, R22.2
- new net N$31: IC2.4, IC4.3
- new net N$32: Q5.B, Q6.C
- net +12V: now also IC4.4, Q5.C, Q6.E
- net GND: now also C7.2, IC4.7, Q7.E, R21.2
Routing:
- net +12V: track 0.00 -> 26.5 mm
- net N$32: track 0.00 -> 11.7 mm
- net N$30: track 0.00 -> 8.53 mm
- net N$28: track 0.00 -> 8.27 mm
- net N$12: track 0.00 -> 5.18 mm
- net N$13: track 0.00 -> 4.20 mm
- net N$26: track 0.00 -> 2.86 mm
Changed lines of the file:
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@@
 <element name="JP4" library="jumper" package="JP4" value="" x="78.74" y="50.8" rot="R180"/>
 <element name="JP6" library="jumper" package="JP4" value="" x="69.85" y="54.61" rot="R90"/>
+<element name="R13" library="resistor" package="M0805" value="" x="5.08" y="58.42" rot="R270"/>
+<element name="IC4" library="burr-brown" package="DIL08" value="OPA336P" x="17.78" y="54.61" rot="R90">
+<attribute name="OC_NEWARK" value="unknown" x="17.78" y="54.61" size="1.778" layer="27" rot="R90" display="off"/>
+<attribute name="MPN" value="" x="17.78" y="54.61" size="1.778" layer="27" rot="R90" display="off"/>
+<attribute name="MF" value="" x="17.78" y="54.61" size="1.778" layer="27" rot="R90" display="off"/>
+<attribute name="OC_FARNELL" value="unknown" x="17.78" y="54.61" size="1.778" layer="27" rot="R90" display="off"/>
+</element>
+<element name="R21" library="resistor" package="M0805" value="" x="19.05" y="52.07" rot="R270"/>
+<element name="R22" library="resistor" package="M0805" value="" x="19.05" y="57.15" rot="R270"/>
+<element name="C7" library="resistor" package="C0805K" value="" x="24.13" y="60.96"/>
+<element name="C8" library="resistor" package="C0805K" value="" x="16.51" y="54.61" rot="R270"/>
+<element name="Q5" library="transistor-power" package="TO220AV" value="TIP41C" x="19.05" y="64.77"/>
+<element name="Q6" library="transistor-power" package="TO220AV" value="TIP42C" x="7.62" y="64.77"/>
+<element name="Q7" library="transistor-npn" package="TO92-EBC" value="BC338" x="10.16" y="55.88" rot="R270"/>
 </elements>
 <signals>
@@
 <contactref element="R19" pad="1"/>
 <contactref element="C6" pad="2"/>
-<wire x1="82.22" y1="69.3" x2="82.28" y2="72.39" width="0" layer="19" extent="1-1"/>
+<contactref element="IC4" pad="7"/>
+<contactref element="R21" pad="2"/>
+<contactref element="C7" pad="2"/>
+<contactref element="Q7" pad="E"/>
+<wire x1="89.62" y1="64.3" x2="92.71" y2="63.77" width="0" layer="19" extent="1-1"/>
+<wire x1="85.42" y1="57.7" x2="89.62" y2="64.3" width="0" layer="19" extent="1-1"/>
+<wire x1="85.36" y1="54.61" x2="85.42" y2="57.7" width="0" layer="19" extent="1-1"/>
+<wire x1="82.22" y1="69.3" x2="89.62" y2="64.3" width="0" layer="19" extent="1-1"/>
+<wire x1="82.28" y1="72.39" x2="82.22" y2="69.3" width="0" layer="19" extent="1-1"/>
 <wire x1="78.02" y1="64.3" x2="82.22" y2="69.3" width="0" layer="19" extent="1-1"/>
 <wire x1="74.93" y1="64.5" x2="78.02" y2="64.3" width="0" layer="19" extent="1-1"/>
-<wire x1="89.62" y1="64.3" x2="82.22" y2="69.3" width="0" layer="19" extent="1-1"/>
-<wire x1="85.42" y1="57.7" x2="89.62" y2="64.3" width="0" layer="19" extent="1-1"/>
-<wire x1="85.36" y1="54.61" x2="85.42" y2="57.7" width="0" layer="19" extent="1-1"/>
-<wire x1="92.71" y1="63.77" x2="89.62" y2="64.3" width="0" layer="19" extent="1-1"/>
-<wire x1="63.5" y1="68.31" x2="85.36" y2="54.61" width="0" layer="19" extent="1-1"/>
+<wire x1="63.5" y1="68.31" x2="74.93" y2="64.5" width="0" layer="19" extent="1-1"/>
 <wire x1="53.34" y1="65.09" x2="63.5" y2="68.31" width="0" layer="19" extent="1-1"/>
 <wire x1="54.61" y1="75.93" x2="53.34" y2="65.09" width="0" layer="19" extent="1-1"/>
-<wire x1="76.52" y1="33.02" x2="92.71" y2="63.77" width="0" layer="19" extent="1-1"/>
+<wire x1="76.52" y1="33.02" x2="85.36" y2="54.61" width="0" layer="19" extent="1-1"/>
 <wire x1="70.17" y1="22.86" x2="76.52" y2="33.02" width="0" layer="19" extent="1-1"/>
 <wire x1="70.17" y1="16.51" x2="70.17" y2="22.86" width="0" layer="19" extent="1-1"/>
@@
 <wire x1="32.385" y1="7.435" x2="33.655" y2="7.435" width="0" layer="19" extent="1-1"/>
 <wire x1="46.67" y1="40.64" x2="57.15" y2="19.05" width="0" layer="19" extent="1-1"/>
+<wire x1="25.13" y1="60.96" x2="53.34" y2="65.09" width="0" layer="19" extent="1-1"/>
+<wire x1="19.05" y1="51.12" x2="25.13" y2="60.96" width="0" layer="19" extent="1-1"/>
+<wire x1="13.97" y1="53.34" x2="19.05" y2="51.12" width="0" layer="19" extent="1-1"/>
+<wire x1="8.89" y1="53.34" x2="13.97" y2="53.34" width="0" layer="19" extent="1-1"/>
 </signal>
 <signal name="+12V">
@@
 <contactref element="IC3" pad="3"/>
 <contactref element="C6" pad="1"/>
+<contactref element="IC4" pad="4"/>
+<contactref element="Q5" pad="C"/>
+<contactref element="Q6" pad="E"/>
+<wire x1="19.05" y1="64.77" x2="22.86" y2="64.77" width="0.4064" layer="1"/>
+<wire x1="22.86" y1="64.77" x2="24.13" y2="63.5" width="0.4064" layer="1"/>
+<wire x1="24.13" y1="63.5" x2="24.13" y2="58.42" width="0.4064" layer="1"/>
+<wire x1="24.13" y1="58.42" x2="21.59" y2="58.42" width="0.4064" layer="1"/>
+<wire x1="19.05" y1="62.23" x2="19.05" y2="64.77" width="0.4064" layer="1"/>
+<wire x1="19.05" y1="64.77" x2="11.43" y2="64.77" width="0.4064" layer="1"/>
+<wire x1="11.43" y1="64.77" x2="10.16" y2="63.5" width="0.4064" layer="1"/>
+<wire x1="10.16" y1="63.5" x2="10.16" y2="62.23" width="0.4064" layer="1"/>
 <wire x1="60.72" y1="66.7" x2="63.5" y2="66.31" width="0" layer="19" extent="1-1"/>
+<wire x1="24.13" y1="63.5" x2="60.72" y2="66.7" width="0" layer="19" extent="1-1"/>
 <wire x1="64.77" y1="24.13" x2="63.5" y2="66.31" width="0" layer="19" extent="1-1"/>
 </signal>
@@
 <contactref element="IC3" pad="4"/>
 <contactref element="R20" pad="2"/>
-<wire x1="81.42" y1="69.3" x2="80.28" y2="72.39" width="0" layer="19" extent="1-1"/>
-<wire x1="74.93" y1="69.53" x2="81.42" y2="69.3" width="0" layer="19" extent="1-1"/>
-<wire x1="78.02" y1="63.5" x2="74.93" y2="69.53" width="0" layer="19" extent="1-1"/>
-<wire x1="74.93" y1="62.5" x2="78.02" y2="63.5" width="0" layer="19" extent="1-1"/>
-<wire x1="89.62" y1="65.1" x2="81.42" y2="69.3" width="0" layer="19" extent="1-1"/>
+<wire x1="89.62" y1="65.1" x2="92.71" y2="65.77" width="0" layer="19" extent="1-1"/>
 <wire x1="86.22" y1="57.7" x2="89.62" y2="65.1" width="0" layer="19" extent="1-1"/>
 <wire x1="87.36" y1="54.61" x2="86.22" y2="57.7" width="0" layer="19" extent="1-1"/>
-<wire x1="92.71" y1="65.77" x2="89.62" y2="65.1" width="0" layer="19" extent="1-1"/>
-<wire x1="58.42" y1="73" x2="87.36" y2="54.61" width="0" layer="19" extent="1-1"/>
+<wire x1="81.42" y1="69.3" x2="89.62" y2="65.1" width="0" layer="19" extent="1-1"/>
+<wire x1="80.28" y1="72.39" x2="81.42" y2="69.3" width="0" layer="19" extent="1-1"/>
+<wire x1="74.93" y1="69.53" x2="80.28" y2="72.39" width="0" layer="19" extent="1-1"/>
+<wire x1="78.02" y1="63.5" x2="81.42" y2="69.3" width="0" layer="19" extent="1-1"/>
+<wire x1="74.93" y1="62.5" x2="78.02" y2="63.5" width="0" layer="19" extent="1-1"/>
+<wire x1="58.42" y1="73" x2="74.93" y2="69.53" width="0" layer="19" extent="1-1"/>
 <wire x1="54.61" y1="73.93" x2="58.42" y2="73" width="0" layer="19" extent="1-1"/>
 <wire x1="53.34" y1="72.07" x2="54.61" y2="73.93" width="0" layer="19" extent="1-1"/>
@@
 <contactref element="IC2" pad="35"/>
 <contactref element="R18" pad="1"/>
-<wire x1="78.02" y1="66.7" x2="74.93" y2="67.63" width="0" layer="19" extent="1-1"/>
+<wire x1="74.93" y1="67.63" x2="78.02" y2="66.7" width="0" layer="19" extent="1-1"/>
 </signal>
 <signal name="N$18">
@@
 <wire x1="53.34" y1="70.17" x2="53.34" y2="66.99" width="0" layer="19" extent="1-1"/>
 </signal>
+<signal name="N$12">
+<contactref element="C7" pad="1"/>
+<contactref element="R22" pad="1"/>
+<contactref element="Q5" pad="E"/>
+<wire x1="21.59" y1="60.96" x2="21.59" y2="62.23" width="0.4064" layer="1"/>
+<wire x1="21.59" y1="60.96" x2="19.05" y2="58.42" width="0.4064" layer="1"/>
+<wire x1="19.05" y1="58.42" x2="19.05" y2="58.1" width="0.4064" layer="1"/>
+<wire x1="21.59" y1="60.96" x2="23.13" y2="60.96" width="0" layer="19" extent="1-1"/>
+</signal>
+<signal name="N$28">
+<contactref element="IC4" pad="6"/>
+<contactref element="C8" pad="1"/>
+<contactref element="Q7" pad="B"/>
+<wire x1="8.89" y1="55.88" x2="13.97" y2="55.88" width="0.4064" layer="16"/>
+<wire x1="13.97" y1="55.88" x2="16.78" y2="55.88" width="0.4064" layer="1"/>
+<wire x1="16.78" y1="55.88" x2="16.51" y2="55.61" width="0.4064" layer="1"/>
+</signal>
+<signal name="N$30">
+<contactref element="IC4" pad="2"/>
+<contactref element="C8" pad="2"/>
+<contactref element="R22" pad="2"/>
+<contactref element="R21" pad="1"/>
+<wire x1="19.05" y1="53.34" x2="21.59" y2="53.34" width="0.4064" layer="1"/>
+<wire x1="19.05" y1="53.34" x2="19.05" y2="56.2" width="0.4064" layer="1"/>
+<wire x1="16.51" y1="53.61" x2="16.51" y2="53.34" width="0.4064" layer="1"/>
+<wire x1="16.51" y1="53.34" x2="19.05" y2="53.34" width="0.4064" layer="1"/>
+<wire x1="19.05" y1="53.34" x2="19.05" y2="53.02" width="0.4064" layer="1"/>
+</signal>
+<signal name="N$31">
+<contactref element="IC2" pad="4"/>
+<contactref element="IC4" pad="3"/>
+<wire x1="21.59" y1="55.88" x2="82.22" y2="57.7" width="0" layer="19" extent="1-1"/>
+</signal>
+<signal name="N$32">
+<contactref element="Q5" pad="B"/>
+<contactref element="Q6" pad="C"/>
+<wire x1="7.62" y1="62.23" x2="7.62" y2="60.96" width="0.4064" layer="1"/>
+<wire x1="7.62" y1="60.96" x2="8.89" y2="59.69" width="0.4064" layer="1"/>
+<wire x1="8.89" y1="59.69" x2="12.7" y2="59.69" width="0.4064" layer="1"/>
+<wire x1="12.7" y1="59.69" x2="15.24" y2="62.23" width="0.4064" layer="1"/>
+<wire x1="15.24" y1="62.23" x2="16.51" y2="62.23" width="0.4064" layer="1"/>
+</signal>
+<signal name="N$13">
+<contactref element="Q7" pad="C"/>
+<contactref element="R13" pad="2"/>
+<wire x1="5.08" y1="57.47" x2="5.4" y2="57.47" width="0.4064" layer="1"/>
+<wire x1="5.4" y1="57.47" x2="6.35" y2="58.42" width="0.4064" layer="1"/>
+<wire x1="6.35" y1="58.42" x2="8.89" y2="58.42" width="0.4064" layer="1"/>
+</signal>
+<signal name="N$26">
+<contactref element="R13" pad="1"/>
+<contactref element="Q6" pad="B"/>
+<wire x1="5.08" y1="59.37" x2="5.08" y2="62.23" width="0.4064" layer="1"/>
+</signal>
 </signals>

Commit message: shrinking
Parts:
- added Q3: BC548, transistor-npn:TO92-EBC
- added Q4: BC557C, transistor-pnp:TO92-EBC
- added Q8: BSS123, transistor-small-signal:SOT23
- added R23, R24, R25, R26, R27, R28, R29, R30: (no value), resistor:0207/2V
- added R31: (no value), resistor:M0805
- C7: value (none) -> 100n
- C8: value (none) -> 100p
- Q1: value BSS92 -> BSS123; device transistor-fet:TO92 -> transistor-small-signal:SOT23
- Q2: value BSS101 -> BSS123; device transistor-fet:TO92 -> transistor-small-signal:SOT23
- R1, R2: device resistor-power:RS02M -> resistor:M0805
- R16, R17: value (none) -> 4R7; device resistor-power:RS02M -> resistor-power:KH208R-8
- R3, R4: value (none) -> 10R; device resistor-power:RS02M -> resistor-power:HPS58
- moved Q1 69.7 mm to (1.27, -3.81), turned to 0 degrees
- moved Q2 69.1 mm to (1.27, -11.4), turned to 0 degrees
- moved R1 67.8 mm to (0.00, -26.7), turned to 0 degrees
- moved R2 66.0 mm to (0.00, -30.5), turned to 0 degrees
- moved R6 35.9 mm to (31.8, 29.2), turned to 180 degrees
- moved R5 33.1 mm to (34.3, 21.6)
- moved IC1 30.5 mm to (31.8, 29.2)
- moved U$1 26.9 mm to (8.89, 19.1)
- moved R4 26.7 mm to (25.4, 25.4)
- moved R3 24.2 mm to (22.9, 27.9)
- moved R10 23.0 mm to (48.3, 21.6)
- moved R7 23.0 mm to (48.3, 25.4)
- moved R8 23.0 mm to (48.3, 27.9)
- moved R9 23.0 mm to (48.3, 19.1)
- moved JP3 23.0 mm to (15.2, 33.0), turned to 90 degrees
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Connections:
- new net N$29: R23.2, R28.2, R29.1, R30.1
- new net N$33: R24.1, R25.1, R26.2, R27.2
- new net N$34: JP3.3, Q3.E, Q4.E
- new net N$35: Q2.3, R2.1, U$1.4
- new net N$36: Q8.3, R1.1, U$2.4
- net +12V: now also R1.2, R2.2, R31.2
- net ADC1: now also R26.1, R27.1; no longer R2.1
- net ADC2: now also R29.2, R30.2; no longer R1.1
- net ADC3: now also R23.1, R28.1; no longer R1.2
- net ADC4: now also R17.1, R24.2, R25.2; no longer R17.2, R2.2
- net GND: now also Q1.2, Q2.2, Q8.2, U$3.1, U$3.2, U$3.3
- net N$16: now also R17.2; no longer R17.1
- net N$6: now also R31.1, U$3.4; no longer JP3.3, Q2.1
- net N$7: now also Q3.C; no longer Q2.3
- net N$8: now also Q4.C; no longer Q1.2
- net N$9: now also Q3.B, Q4.B; no longer Q1.1, Q2.2
Routing:
- net N$6: track 46.1 -> 0.00 mm
- net N$1: track 47.1 -> 8.17 mm
- net ADC1: track 46.7 -> 25.3 mm
- net ADC2: track 35.2 -> 17.9 mm
- net ADC4: track 0.00 -> 16.9 mm
- net N$29: track 0.00 -> 12.7 mm
- net N$34: track 0.00 -> 11.2 mm
- net N$7: track 13.6 -> 2.54 mm
- net N$14: track 0.00 -> 10.7 mm
- net N$33: track 0.00 -> 9.72 mm
- net N$11: track 4.98 -> 13.5 mm
- net N$16: track 0.00 -> 6.13 mm
- net N$15: track 0.00 -> 5.08 mm
- net N$4: track 11.5 -> 7.38 mm
- net N$8: track 6.13 -> 2.54 mm
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